File: ina260.kicad_sch (KiCad schematic)
At the start: 2 parts, among them U2 INA260AIPWR

Commit message: Initial entry
Parts:
- renumbered U2 to U3
Changed lines of the file:
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@@
 		(instances
 			(project "TrailerMonitor"
-				(path "/3e352327-6d34-4520-89b7-9902d021830c/15758eaf-da29-4bf9-824e-05489805e872"
-					(reference "C5")
-					(unit 1)
-				)
-				(path "/3e352327-6d34-4520-89b7-9902d021830c/2a394739-6618-41e7-ac02-7d9ae9b51130"
-					(reference "C7")
-					(unit 1)
-				)
-				(path "/3e352327-6d34-4520-89b7-9902d021830c/3f450dac-4b40-43e0-a03c-1caf434b0aa7"
-					(reference "C4")
-					(unit 1)
-				)
-				(path "/3e352327-6d34-4520-89b7-9902d021830c/791c4b70-f492-4b91-a1f1-088e70f1a198"
-					(reference "C3")
-					(unit 1)
-				)
-				(path "/3e352327-6d34-4520-89b7-9902d021830c/8d32305e-b711-49b4-8873-054d0245a6aa"
-					(reference "C6")
-					(unit 1)
-				)
-				(path "/3e352327-6d34-4520-89b7-9902d021830c/99793f99-a72e-458a-aafa-ed725c74b251"
-					(reference "C8")
-					(unit 1)
-				)
-				(path "/3e352327-6d34-4520-89b7-9902d021830c/9d259bb6-46c1-4cbd-90bb-8c019a72ebc4"
-					(reference "C2")
-					(unit 1)
-				)
 				(path "/3e352327-6d34-4520-89b7-9902d021830c/d8c4f0ea-7758-4aba-8b6e-91a4eea3fbe2"
 					(reference "C1")
@@
 		(instances
 			(project "TrailerMonitor"
-				(path "/3e352327-6d34-4520-89b7-9902d021830c/15758eaf-da29-4bf9-824e-05489805e872"
-					(reference "#PWR010")
-					(unit 1)
-				)
-				(path "/3e352327-6d34-4520-89b7-9902d021830c/2a394739-6618-41e7-ac02-7d9ae9b51130"
-					(reference "#PWR014")
-					(unit 1)
-				)
-				(path "/3e352327-6d34-4520-89b7-9902d021830c/3f450dac-4b40-43e0-a03c-1caf434b0aa7"
-					(reference "#PWR08")
-					(unit 1)
-				)
-				(path "/3e352327-6d34-4520-89b7-9902d021830c/791c4b70-f492-4b91-a1f1-088e70f1a198"
-					(reference "#PWR06")
-					(unit 1)
-				)
-				(path "/3e352327-6d34-4520-89b7-9902d021830c/8d32305e-b711-49b4-8873-054d0245a6aa"
-					(reference "#PWR012")
-					(unit 1)
-				)
-				(path "/3e352327-6d34-4520-89b7-9902d021830c/99793f99-a72e-458a-aafa-ed725c74b251"
-					(reference "#PWR016")
-					(unit 1)
-				)
-				(path "/3e352327-6d34-4520-89b7-9902d021830c/9d259bb6-46c1-4cbd-90bb-8c019a72ebc4"
-					(reference "#PWR04")
-					(unit 1)
-				)
 				(path "/3e352327-6d34-4520-89b7-9902d021830c/d8c4f0ea-7758-4aba-8b6e-91a4eea3fbe2"
 					(reference "#PWR02")
@@
 		(dnp no)
 		(fields_autoplaced yes)
-		(property "Reference" "U2"
+		(property "Reference" "U3"
 			(at 147.32 73.66 0)
 			(show_name no)
@@
 		(instances
 			(project "TrailerMonitor"
-				(path "/3e352327-6d34-4520-89b7-9902d021830c/15758eaf-da29-4bf9-824e-05489805e872"
-					(reference "U6")
-					(unit 1)
-				)
-				(path "/3e352327-6d34-4520-89b7-9902d021830c/2a394739-6618-41e7-ac02-7d9ae9b51130"
-					(reference "U8")
-					(unit 1)
-				)
-				(path "/3e352327-6d34-4520-89b7-9902d021830c/3f450dac-4b40-43e0-a03c-1caf434b0aa7"
-					(reference "U5")
-					(unit 1)
-				)
-				(path "/3e352327-6d34-4520-89b7-9902d021830c/791c4b70-f492-4b91-a1f1-088e70f1a198"
-					(reference "U4")
-					(unit 1)
-				)
-				(path "/3e352327-6d34-4520-89b7-9902d021830c/8d32305e-b711-49b4-8873-054d0245a6aa"
-					(reference "U7")
-					(unit 1)
-				)
-				(path "/3e352327-6d34-4520-89b7-9902d021830c/99793f99-a72e-458a-aafa-ed725c74b251"
-					(reference "U9")
-					(unit 1)
-				)
-				(path "/3e352327-6d34-4520-89b7-9902d021830c/9d259bb6-46c1-4cbd-90bb-8c019a72ebc4"
+				(path "/3e352327-6d34-4520-89b7-9902d021830c/d8c4f0ea-7758-4aba-8b6e-91a4eea3fbe2"
 					(reference "U3")
-					(unit 1)
-				)
-				(path "/3e352327-6d34-4520-89b7-9902d021830c/d8c4f0ea-7758-4aba-8b6e-91a4eea3fbe2"
-					(reference "U2")
 					(unit 1)
 				)
@@
 		(instances
 			(project "TrailerMonitor"
-				(path "/3e352327-6d34-4520-89b7-9902d021830c/15758eaf-da29-4bf9-824e-05489805e872"
-					(reference "#PWR09")
-					(unit 1)
-				)
-				(path "/3e352327-6d34-4520-89b7-9902d021830c/2a394739-6618-41e7-ac02-7d9ae9b51130"
-					(reference "#PWR013")
-					(unit 1)
-				)
-				(path "/3e352327-6d34-4520-89b7-9902d021830c/3f450dac-4b40-43e0-a03c-1caf434b0aa7"
-					(reference "#PWR07")
-					(unit 1)
-				)
-				(path "/3e352327-6d34-4520-89b7-9902d021830c/791c4b70-f492-4b91-a1f1-088e70f1a198"
-					(reference "#PWR05")
-					(unit 1)
-				)
-				(path "/3e352327-6d34-4520-89b7-9902d021830c/8d32305e-b711-49b4-8873-054d0245a6aa"
-					(reference "#PWR011")
-					(unit 1)
-				)
-				(path "/3e352327-6d34-4520-89b7-9902d021830c/99793f99-a72e-458a-aafa-ed725c74b251"
-					(reference "#PWR015")
-					(unit 1)
-				)
-				(path "/3e352327-6d34-4520-89b7-9902d021830c/9d259bb6-46c1-4cbd-90bb-8c019a72ebc4"
-					(reference "#PWR03")
-					(unit 1)
-				)
 				(path "/3e352327-6d34-4520-89b7-9902d021830c/d8c4f0ea-7758-4aba-8b6e-91a4eea3fbe2"
 					(reference "#PWR01")

Commit message: Initial layout; remove INA260
Parts:
- C6: renamed from C1; footprint Capacitor_SMD:C_0805_2012Metric -> Capacitor_SMD:C_1206_3216Metric
- renumbered U3 to U4
Changed lines of the file:
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@@
 	(title_block
 		(title "Trailer Monitor")
-		(date "2025-09-20")
-		(rev "V1.0")
+		(date "2026-08-30")
+		(rev "V1.1")
 		(company "Tripoli Central Virginia")
 	)
@@
 		(dnp no)
 		(fields_autoplaced yes)
-		(property "Reference" "C1"
+		(property "Reference" "C6"
 			(at 111.76 76.2064 90)
 			(show_name no)
@@
 			)
 		)
-		(property "Footprint" "Capacitor_SMD:C_0805_2012Metric"
+		(property "Footprint" "Capacitor_SMD:C_1206_3216Metric"
 			(at 118.11 76.2 0)
 			(hide yes)
@@
 			(project "TrailerMonitor"
 				(path "/3e352327-6d34-4520-89b7-9902d021830c/d8c4f0ea-7758-4aba-8b6e-91a4eea3fbe2"
-					(reference "C1")
+					(reference "C6")
 					(unit 1)
 				)
@@
 		(dnp no)
 		(fields_autoplaced yes)
-		(property "Reference" "#PWR02"
+		(property "Reference" "#PWR025"
 			(at 166.37 121.92 0)
 			(hide yes)
@@
 			(project "TrailerMonitor"
 				(path "/3e352327-6d34-4520-89b7-9902d021830c/d8c4f0ea-7758-4aba-8b6e-91a4eea3fbe2"
-					(reference "#PWR02")
+					(reference "#PWR025")
 					(unit 1)
 				)
@@
 		(dnp no)
 		(fields_autoplaced yes)
-		(property "Reference" "U3"
+		(property "Reference" "U4"
 			(at 147.32 73.66 0)
 			(show_name no)
@@
 			(project "TrailerMonitor"
 				(path "/3e352327-6d34-4520-89b7-9902d021830c/d8c4f0ea-7758-4aba-8b6e-91a4eea3fbe2"
-					(reference "U3")
+					(reference "U4")
 					(unit 1)
 				)
@@
 		(dnp no)
 		(fields_autoplaced yes)
-		(property "Reference" "#PWR01"
+		(property "Reference" "#PWR024"
 			(at 118.11 63.5 0)
 			(hide yes)
@@
 			(project "TrailerMonitor"
 				(path "/3e352327-6d34-4520-89b7-9902d021830c/d8c4f0ea-7758-4aba-8b6e-91a4eea3fbe2"
-					(reference "#PWR01")
+					(reference "#PWR024")
 					(unit 1)
 				)
