File: TrailerMonitor.kicad_pcb (KiCad board)
At the start: 2 copper layers, 69 x 53.8 mm, 22 parts, among them J1 +VIN (7-60 VDC), J2 ModBus, J3 LED (Power), J4 LED (ModBus Act), Q1 DMG2305UX-13, U1 MAX485ESA+, U2 LMR51606XDBVR

Commit message: Add OLED display, remove ModBus ACT LED
Parts:
- removed J4: LED (ModBus Act), Connector_Molex:Molex_KK-254_AE-6410-02A_1x02_P2.54mm_Vertical
- removed R4: 160, Resistor_SMD:R_0805_2012Metric
- added J5: OLED Display, Connector_Molex:Molex_KK-254_AE-6410-04A_1x04_P2.54mm_Vertical, F.Cu at (134.8, 93.9)
- J2: value ModBus -> Conn_01x04; footprint Connector_Molex:Molex_KK-254_AE-6410-02A_1x02_P2.54mm_Vertical -> Connector_Molex:Molex_KK-254_AE-6410-04A_1x04_P2.54mm_Vertical
- moved J3 53.2 mm to (134.8, 107.6), turned to 90 degrees
- moved R3 47.0 mm to (134.8, 101.1), turned to 90 degrees
- moved J2 3.94 mm to (187.3, 98.7)
- moved J1 2.36 mm to (187.3, 90.0)
Connections:
- A1 pad 29: /MODBUS_ACT -> unconnected-(A1-GPIO22-Pad29)
- A1 pad 4: unconnected-(A1-GPIO2-Pad4) -> /SDA
- A1 pad 5: unconnected-(A1-GPIO3-Pad5) -> /SCL
- J2 pad 1: /B -> +5V
- J2 pad 2: /A -> /B
Routing:
- net /MODBUS_ACT: track 33.0 -> 0.00 mm
- net /SDA: track 0.00 -> 9.59 mm
- net /SCL: track 0.00 -> 9.39 mm
- net Net-(J4-Pin_2): track 5.16 -> 0.00 mm
- net /A: track 18.0 -> 15.0 mm
- net /B: track 18.5 -> 15.9 mm
- net Net-(J3-Pin_2): track 5.36 -> 3.00 mm
- net Net-(J1-Pin_1): track 15.2 -> 15.9 mm
- net +5V: vias 5 -> 9
Other:
- board text added: "OLED DISPLAY"
- board text added: "TRAILER MONITOR V1.1 MIKE McPHERSON 2026"
- board text removed: "MODBUS ACT LED"
- board text removed: "TRAILER MONITOR V1.0 MIKE McPHERSON"
